Commit message: Properly use calibration xacro file

File: hector_tracker_description/calibrations/spinning_lidar_calibration.urdf.xacro (robot description, xacro)
@@ -6,4 +6,4 @@
 <!-- =================================================================================== -->
 <robot xmlns:xacro="http://www.ros.org/wiki/xacro" name="calibration">
-  <origin rpy="0.0 0.0 0.0" xyz="0.0 0.0 0.0"/>
+  <origin xyz="-0.025 0.0 0.0" rpy="0.0 ${M_PI*0.75} 0.0"/>
 </robot>
