Commit message: Remove stabilized lidar for the moment

File: hector_tracker_description/urdf/tracker_default.urdf.xacro (robot description, xacro)
@@ -75,4 +75,5 @@
     </plugin>
   </gazebo>
+  <!--
   <joint name="stab_laser_roll_joint" type="revolute">
     <origin xyz="${-0.26} 0.1 ${0.43}" rpy="0 0 0"/>
@@ -110,5 +111,5 @@
       <origin xyz="0.0 0.0 ${laser1_size_z/2}" rpy="0 0 0"/>
       <geometry>
-        <!--<box size="${laser1_size_x} ${laser1_size_y} ${laser1_size_z}" />-->
+        <!+-<box size="${laser1_size_x} ${laser1_size_y} ${laser1_size_z}" /> ->
         <box size="${laser1_size_x} ${laser1_size_y} 0.01"/>
       </geometry>
@@ -118,5 +119,5 @@
       <origin xyz="0.0 0.0 ${laser1_size_z/2}" rpy="0 0 0"/>
       <geometry>
-        <!--<box size="${laser1_size_x} ${laser1_size_y} ${laser1_size_z}" />-->
+        <!+-<box size="${laser1_size_x} ${laser1_size_y} ${laser1_size_z}" />->
         <box size="${laser1_size_x} ${laser1_size_y} 0.01"/>
       </geometry>
@@ -131,4 +132,8 @@
   <xacro:joint_standard_transmission name="stab_laser_roll_joint"/>
   <xacro:joint_standard_transmission name="stab_laser_pitch_joint"/>
+  <xacro:hokuyo_utm30lx name="stab_laser" parent="stab_laser_pitch_link" ros_topic="/stab_laser/scan_gazebo" update_rate="40" ray_count="1081" min_angle="135" max_angle="-135">
+    <origin xyz="${laser1_center_x_offset} 0 ${laser1_plane_height}" rpy="0 0 0"/>
+  </xacro:hokuyo_utm30lx>
+  -->
   <gazebo>
     <!-- ros_control plugin -->
@@ -170,7 +175,4 @@
     <origin xyz="${kinect_x_position} ${kinect_y_position}  ${0.035}" rpy="${kinect_roll_position} ${kinect_pitch_position} ${kinect_yaw_position}"/>
   </xacro:realsense_camera>
-  <xacro:hokuyo_utm30lx name="stab_laser" parent="stab_laser_pitch_link" ros_topic="/stab_laser/scan_gazebo" update_rate="40" ray_count="1081" min_angle="135" max_angle="-135">
-    <origin xyz="${laser1_center_x_offset} 0 ${laser1_plane_height}" rpy="0 0 0"/>
-  </xacro:hokuyo_utm30lx>
   <!-- <xacro:vision_box_common_gazebo_plugins/> -->
   <xacro:include filename="$(find hector_tracker_description)/urdf/tracker_spinning_lidar_mount.urdf.xacro.xml" />

Commit message: Update structure addons

File: hector_tracker_description/urdf/tracker_default.urdf.xacro (robot description, xacro)
@@ -144,5 +144,5 @@
   </gazebo>
   <joint name="structure_addon_joint" type="fixed">
-    <origin xyz="${-0.275} 0.1 ${0.3}" rpy="0 0 0"/>
+    <origin xyz="0 0 ${0.185}" rpy="0 0 0"/>
     <parent link="base_link"/>
     <child link="structure_addons_link"/>
@@ -150,5 +150,5 @@
   <link name="structure_addons_link">
     <xacro:inertial_cube mass="0.1" diameter="0.07"/>
-    <visual>
+    <!--<visual>
       <origin xyz="-0.0 0.0 0.0" rpy="0 0 0"/>
       <geometry>
@@ -163,4 +163,36 @@
       <geometry>
         <box size="0.20 0.1 0.2"/>
+      </geometry>
+    </collision>
+    -->
+    <!--Lowest box-->
+    <visual>
+      <origin xyz="${-0.29.5} 0.115 ${0.115/2}" rpy="0 0 0"/>
+      <geometry>
+        <box size="${0.43-0.16} 0.15 0.115"/>
+      </geometry>
+    </visual>
+    <!--Middle box-->
+    <visual>
+      <origin xyz="${-0.34} 0.115 ${0.115+0.25*0.5}" rpy="0 0 0"/>
+      <geometry>
+        <box size="${0.43-0.25} 0.15 0.25"/>
+      </geometry>
+    </visual>
+    <!--
+    40.8 from ref point to back of alum. frame - 12.3 (11.7 to 12.9 rotation shaft)
+    27.6 to top of alum. platform + 16.6 for lidar center
+    -->
+    <!--Antenna-->
+    <visual>
+      <origin xyz="${-0.38} -0.175 0.11" rpy="0 0 0"/>
+      <geometry>
+        <cylinder radius="0.015" length="0.22" />
+      </geometry>
+    </visual>
+    <collision>
+      <origin xyz="${-0.38} -0.175 0.11" rpy="0 0 0"/>
+      <geometry>
+        <cylinder radius="0.0175" length="0.22" />
       </geometry>
     </collision>
@@ -178,5 +210,5 @@
   <xacro:include filename="$(find hector_tracker_description)/urdf/tracker_spinning_lidar_mount.urdf.xacro.xml" />
   <xacro:tracker_spinning_lidar_mount_macro parent="base_link"  name="spin_lidar" scaling="0.001">
-    <origin xyz="-0.3 0.1 0.58" rpy="0.0 ${-M_PI*0.5} ${M_PI}"/>
+    <origin xyz="-0.285 0.1 0.627" rpy="0.0 ${-M_PI*0.5} ${M_PI}"/>
     <origin xyz="0 0.0 0.0" rpy="0.0 ${M_PI*0.75} 0.0"/>
   </xacro:tracker_spinning_lidar_mount_macro>

Commit message: Updated sensor head measures

File: hector_tracker_description/urdf/tracker_default.urdf.xacro (robot description, xacro)
@@ -27,5 +27,5 @@
   <xacro:include filename="$(find hector_components_description)/urdf/vision_box_dimensions_hector2.urdf.xacro" />
   <joint name="sensor_head_yaw_joint" type="revolute">
-    <origin xyz="-0.01 ${0.04} 0.075" rpy="0 0 0"/>
+    <origin xyz="-0.03 ${0.0565} 0.089" rpy="0 0 0"/>
     <parent link="arm_link_3"/>
     <child link="sensor_head_yaw_link"/>
@@ -50,8 +50,8 @@
   </link>
   <joint name="sensor_head_pitch_joint" type="revolute">
-    <origin xyz="0 0 ${cameraYawServo_size_z}" rpy="0 0 0"/>
+    <origin xyz="0 -0.0235 0.0921" rpy="${-M_PI/2} 0 0"/>
     <parent link="sensor_head_yaw_link"/>
     <child link="sensor_head_mount_link"/>
-    <axis xyz="0 1 0"/>
+    <axis xyz="0 0 1"/>
     <limit lower="${-M_PI/2}" upper="${M_PI/2}" effort="100" velocity="100"/>
   </joint>
@@ -202,8 +202,9 @@
   </gazebo>
   <xacro:flir_a35_camera name="arm_thermal_cam" parent="sensor_head_mount_link">
-    <origin xyz="${infrared_x_position} ${infrared_y_position} ${infrared_z_position}" rpy="0 0 0"/>
+    <!--origin xyz="${infrared_x_position} ${infrared_y_position} ${infrared_z_position}" rpy="0 0 0"/-->
+    <origin xyz="0.0345 0.0 -0.03106" rpy="0 0 0"/>
   </xacro:flir_a35_camera>
   <xacro:realsense_camera name="arm_rgbd_cam" parent="sensor_head_mount_link">
-    <origin xyz="${kinect_x_position} ${kinect_y_position}  ${0.035}" rpy="${kinect_roll_position} ${kinect_pitch_position} ${kinect_yaw_position}"/>
+    <origin xyz="0.01 -0.048  0.01373" rpy="${M_PI*0.5} ${kinect_pitch_position} ${kinect_yaw_position}"/>
   </xacro:realsense_camera>
   <!-- <xacro:vision_box_common_gazebo_plugins/> -->

Commit message: Added collision geometry to structure addons

File: hector_tracker_description/urdf/tracker_default.urdf.xacro (robot description, xacro)
@@ -173,4 +173,10 @@
       </geometry>
     </visual>
+    <collision>
+      <origin xyz="${-0.29.5} 0.115 ${0.115/2}" rpy="0 0 0"/>
+      <geometry>
+        <box size="${0.43-0.16} 0.15 0.115"/>
+      </geometry>
+    </collision>
     <!--Middle box-->
     <visual>
@@ -180,4 +186,10 @@
       </geometry>
     </visual>
+    <collision>
+      <origin xyz="${-0.34} 0.115 ${0.115+0.25*0.5}" rpy="0 0 0"/>
+      <geometry>
+        <box size="${0.43-0.25} 0.15 0.25"/>
+      </geometry>
+    </collision>
     <!--
     40.8 from ref point to back of alum. frame - 12.3 (11.7 to 12.9 rotation shaft)

Commit message: Increased height of structure addons to avoid collisions with gps module

File: hector_tracker_description/urdf/tracker_default.urdf.xacro (robot description, xacro)
@@ -181,13 +181,13 @@
     <!--Middle box-->
     <visual>
-      <origin xyz="${-0.34} 0.115 ${0.115+0.25*0.5}" rpy="0 0 0"/>
-      <geometry>
-        <box size="${0.43-0.25} 0.15 0.25"/>
-      </geometry>
-    </visual>
-    <collision>
-      <origin xyz="${-0.34} 0.115 ${0.115+0.25*0.5}" rpy="0 0 0"/>
-      <geometry>
-        <box size="${0.43-0.25} 0.15 0.25"/>
+      <origin xyz="${-0.34} 0.115 ${0.215+0.25*0.5}" rpy="0 0 0"/>
+      <geometry>
+        <box size="${0.43-0.25} 0.15 0.45"/>
+      </geometry>
+    </visual>
+    <collision>
+      <origin xyz="${-0.34} 0.115 ${0.215+0.25*0.5}" rpy="0 0 0"/>
+      <geometry>
+        <box size="${0.43-0.25} 0.15 0.45"/>
       </geometry>
     </collision>

Commit message: offset for spinning lidar corrected

File: hector_tracker_description/urdf/tracker_default.urdf.xacro (robot description, xacro)
@@ -223,5 +223,5 @@
   <xacro:include filename="$(find hector_tracker_description)/urdf/tracker_spinning_lidar_mount.urdf.xacro.xml" />
   <xacro:tracker_spinning_lidar_mount_macro parent="base_link"  name="spin_lidar" scaling="0.001">
-    <origin xyz="-0.285 0.1 0.627" rpy="0.0 ${-M_PI*0.5} ${M_PI}"/>
+    <origin xyz="-0.285 0.1 0.627" rpy="0.0 ${-M_PI*0.5} ${M_PI-0.75}"/>
     <origin xyz="0 0.0 0.0" rpy="0.0 ${M_PI*0.75} 0.0"/>
   </xacro:tracker_spinning_lidar_mount_macro>

Commit message: Lidar position corrected

File: hector_tracker_description/urdf/tracker_default.urdf.xacro (robot description, xacro)
@@ -223,6 +223,6 @@
   <xacro:include filename="$(find hector_tracker_description)/urdf/tracker_spinning_lidar_mount.urdf.xacro.xml" />
   <xacro:tracker_spinning_lidar_mount_macro parent="base_link"  name="spin_lidar" scaling="0.001">
-    <origin xyz="-0.285 0.1 0.627" rpy="0.0 ${-M_PI*0.5} ${M_PI-0.75}"/>
-    <origin xyz="0 0.0 0.0" rpy="0.0 ${M_PI*0.75} 0.0"/>
+    <origin xyz="-0.285 0.14 0.627" rpy="0.0 ${-M_PI*0.5} ${M_PI-0.75}"/>
+    <origin xyz="-0.025 0.0 0.0" rpy="0.0 ${M_PI*0.75} 0.0"/>
   </xacro:tracker_spinning_lidar_mount_macro>
   <gazebo>

Commit message: Spin lidar orientation ajusted

File: hector_tracker_description/urdf/tracker_default.urdf.xacro (robot description, xacro)
@@ -223,5 +223,5 @@
   <xacro:include filename="$(find hector_tracker_description)/urdf/tracker_spinning_lidar_mount.urdf.xacro.xml" />
   <xacro:tracker_spinning_lidar_mount_macro parent="base_link"  name="spin_lidar" scaling="0.001">
-    <origin xyz="-0.285 0.14 0.627" rpy="0.0 ${-M_PI*0.5} ${M_PI-0.75}"/>
+    <origin xyz="-0.285 0.14 0.627" rpy="0.05 ${-M_PI*0.485} ${M_PI-0.75}"/>
     <origin xyz="-0.025 0.0 0.0" rpy="0.0 ${M_PI*0.75} 0.0"/>
   </xacro:tracker_spinning_lidar_mount_macro>

Commit message: Move realsense due to how updated macro works

File: hector_tracker_description/urdf/tracker_default.urdf.xacro (robot description, xacro)
@@ -218,5 +218,5 @@
   </xacro:flir_a35_camera>
   <xacro:realsense_camera name="arm_rgbd_cam" parent="sensor_head_mount_link">
-    <origin xyz="0.01 -0.048  0.01373" rpy="${M_PI*0.5} ${kinect_pitch_position} ${kinect_yaw_position}"/>
+    <origin xyz="0.01 -0.048  ${0.01373-0.051}" rpy="${M_PI*0.5} ${kinect_pitch_position} ${kinect_yaw_position}"/>
   </xacro:realsense_camera>
   <!-- <xacro:vision_box_common_gazebo_plugins/> -->

Commit message: Added stabilized lidar

File: hector_tracker_description/urdf/tracker_default.urdf.xacro (robot description, xacro)
@@ -75,8 +75,7 @@
     </plugin>
   </gazebo>
-  <!--
   <joint name="stab_laser_roll_joint" type="revolute">
-    <origin xyz="${-0.26} 0.1 ${0.43}" rpy="0 0 0"/>
-    <parent link="base_link"/>
+    <origin xyz="${-0.007} -0.046 ${0.078}" rpy="0 0 ${-M_PI/2}"/>
+    <parent link="arm_link_0"/>
     <child link="stab_laser_roll_link"/>
     <axis xyz="1 0 0"/>
@@ -111,5 +110,5 @@
       <origin xyz="0.0 0.0 ${laser1_size_z/2}" rpy="0 0 0"/>
       <geometry>
-        <!+-<box size="${laser1_size_x} ${laser1_size_y} ${laser1_size_z}" /> ->
+        <!--<box size="${laser1_size_x} ${laser1_size_y} ${laser1_size_z}" /> -->
         <box size="${laser1_size_x} ${laser1_size_y} 0.01"/>
       </geometry>
@@ -119,5 +118,5 @@
       <origin xyz="0.0 0.0 ${laser1_size_z/2}" rpy="0 0 0"/>
       <geometry>
-        <!+-<box size="${laser1_size_x} ${laser1_size_y} ${laser1_size_z}" />->
+        <!--<box size="${laser1_size_x} ${laser1_size_y} ${laser1_size_z}" />-->
         <box size="${laser1_size_x} ${laser1_size_y} 0.01"/>
       </geometry>
@@ -135,5 +134,4 @@
     <origin xyz="${laser1_center_x_offset} 0 ${laser1_plane_height}" rpy="0 0 0"/>
   </xacro:hokuyo_utm30lx>
-  -->
   <gazebo>
     <!-- ros_control plugin -->

Commit message: Added stabilized lidar (reverted from commit e4f42a0391cf3aa35818884e2d96644b22dba529)

File: hector_tracker_description/urdf/tracker_default.urdf.xacro (robot description, xacro)
@@ -75,7 +75,8 @@
     </plugin>
   </gazebo>
+  <!--
   <joint name="stab_laser_roll_joint" type="revolute">
-    <origin xyz="${-0.007} -0.046 ${0.078}" rpy="0 0 ${-M_PI/2}"/>
-    <parent link="arm_link_0"/>
+    <origin xyz="${-0.26} 0.1 ${0.43}" rpy="0 0 0"/>
+    <parent link="base_link"/>
     <child link="stab_laser_roll_link"/>
     <axis xyz="1 0 0"/>
@@ -110,5 +111,5 @@
       <origin xyz="0.0 0.0 ${laser1_size_z/2}" rpy="0 0 0"/>
       <geometry>
-        <!--<box size="${laser1_size_x} ${laser1_size_y} ${laser1_size_z}" /> -->
+        <!+-<box size="${laser1_size_x} ${laser1_size_y} ${laser1_size_z}" /> ->
         <box size="${laser1_size_x} ${laser1_size_y} 0.01"/>
       </geometry>
@@ -118,5 +119,5 @@
       <origin xyz="0.0 0.0 ${laser1_size_z/2}" rpy="0 0 0"/>
       <geometry>
-        <!--<box size="${laser1_size_x} ${laser1_size_y} ${laser1_size_z}" />-->
+        <!+-<box size="${laser1_size_x} ${laser1_size_y} ${laser1_size_z}" />->
         <box size="${laser1_size_x} ${laser1_size_y} 0.01"/>
       </geometry>
@@ -134,4 +135,5 @@
     <origin xyz="${laser1_center_x_offset} 0 ${laser1_plane_height}" rpy="0 0 0"/>
   </xacro:hokuyo_utm30lx>
+  -->
   <gazebo>
     <!-- ros_control plugin -->

Commit message: added pseyes

File: hector_tracker_description/urdf/tracker_default.urdf.xacro (robot description, xacro)
@@ -231,4 +231,10 @@
     </plugin>
   </gazebo>
+    <xacro:generic_camera name="pseye_left_cam" parent="base_link" ros_topic="image_raw" cam_info_topic="camera_info" update_rate="10" res_x="640" res_y="480" image_format="R8G8B8" hfov="120">
+    <origin xyz="${-0.285-0.17} ${0.14+0.05} ${0.627-0.11}" rpy="0 0 2.35619"/>
+  </xacro:generic_camera>
+  <xacro:generic_camera name="pseye_right_cam" parent="base_link" ros_topic="image_raw" cam_info_topic="camera_info" update_rate="10" res_x="640" res_y="480" image_format="R8G8B8" hfov="120">
+    <origin xyz="${-0.285-0.17} ${0.14-0.05} ${0.627-0.11}" rpy="0 0 -2.35619"/>
+  </xacro:generic_camera> -->
   <xacro:generic_camera name="front_chassis_cam" parent="base_link" ros_topic="image_raw" cam_info_topic="camera_info" update_rate="10" res_x="640" res_y="480" image_format="R8G8B8" hfov="120">
     <origin xyz="${0.1+0.122} 0.0 0.11" rpy="0 0 0"/>

Commit message: spin lidar offset adjusted

File: hector_tracker_description/urdf/tracker_default.urdf.xacro (robot description, xacro)
@@ -221,5 +221,5 @@
   <xacro:include filename="$(find hector_tracker_description)/urdf/tracker_spinning_lidar_mount.urdf.xacro.xml" />
   <xacro:tracker_spinning_lidar_mount_macro parent="base_link"  name="spin_lidar" scaling="0.001">
-    <origin xyz="-0.285 0.14 0.627" rpy="0.05 ${-M_PI*0.485} ${M_PI-0.75}"/>
+    <origin xyz="-0.285 0.14 0.627" rpy="0.05 ${-M_PI*0.485} ${M_PI-0.61}"/>
     <origin xyz="-0.025 0.0 0.0" rpy="0.0 ${M_PI*0.75} 0.0"/>
   </xacro:tracker_spinning_lidar_mount_macro>

Commit message: offset adjusted

File: hector_tracker_description/urdf/tracker_default.urdf.xacro (robot description, xacro)
@@ -221,5 +221,5 @@
   <xacro:include filename="$(find hector_tracker_description)/urdf/tracker_spinning_lidar_mount.urdf.xacro.xml" />
   <xacro:tracker_spinning_lidar_mount_macro parent="base_link"  name="spin_lidar" scaling="0.001">
-    <origin xyz="-0.285 0.14 0.627" rpy="0.05 ${-M_PI*0.485} ${M_PI-0.61}"/>
+    <origin xyz="-0.285 0.14 0.627" rpy="0.05 ${-M_PI*0.485} ${M_PI-1.2}"/>
     <origin xyz="-0.025 0.0 0.0" rpy="0.0 ${M_PI*0.75} 0.0"/>
   </xacro:tracker_spinning_lidar_mount_macro>

Commit message: Adjust lidar offset

File: hector_tracker_description/urdf/tracker_default.urdf.xacro (robot description, xacro)
@@ -221,5 +221,5 @@
   <xacro:include filename="$(find hector_tracker_description)/urdf/tracker_spinning_lidar_mount.urdf.xacro.xml" />
   <xacro:tracker_spinning_lidar_mount_macro parent="base_link"  name="spin_lidar" scaling="0.001">
-    <origin xyz="-0.285 0.14 0.627" rpy="0.05 ${-M_PI*0.485} ${M_PI-1.2}"/>
+    <origin xyz="-0.285 0.14 0.627" rpy="0.05 ${-M_PI*0.485} ${M_PI-0.9}"/>
     <origin xyz="-0.025 0.0 0.0" rpy="0.0 ${M_PI*0.75} 0.0"/>
   </xacro:tracker_spinning_lidar_mount_macro>

Commit message: Add navsat link and associated gazebo plugin

File: hector_tracker_description/urdf/tracker_default.urdf.xacro (robot description, xacro)
@@ -211,4 +211,36 @@
     <material>Gazebo/Grey</material>
   </gazebo>
+    <!-- TODO: Same note as applies to imu_link -->
+  <link name="navsat_link">
+    <!--
+    <visual>
+      <geometry>
+        <cylinder radius="0.026" length="0.016" />
+      </geometry>
+      <origin xyz="0 0 0.008" />
+      <material name="black" />
+    </visual>
+    -->
+  </link>
+  <joint name="navsat_joint" type="fixed">
+    <parent link="base_link" />
+    <child link="navsat_link" />
+    <origin xyz="${-0.35.5} 0.115 ${0.68}" rpy="0 0 0"/>
+  </joint>
+  <gazebo>
+    <plugin name="gps_controller" filename="libhector_gazebo_ros_gps.so">
+      <updateRate>5</updateRate>
+      <robotNamespace>/</robotNamespace>
+      <bodyName>navsat_link</bodyName>
+      <frameId>base_link</frameId>
+      <topicName>/navsat/fix</topicName>
+      <velocityTopicName>/navsat/vel</velocityTopicName>
+      <referenceLatitude>49.9</referenceLatitude>
+      <referenceLongitude>8.9</referenceLongitude>
+      <referenceHeading>0</referenceHeading>
+      <referenceAltitude>0</referenceAltitude>
+      <drift>0.0001 0.0001 0.0001</drift>
+    </plugin>
+  </gazebo>
   <xacro:flir_a35_camera name="arm_thermal_cam" parent="sensor_head_mount_link">
     <!--origin xyz="${infrared_x_position} ${infrared_y_position} ${infrared_z_position}" rpy="0 0 0"/-->

Commit message: Correct orientation for thermal cam

File: hector_tracker_description/urdf/tracker_default.urdf.xacro (robot description, xacro)
@@ -245,5 +245,5 @@
   <xacro:flir_a35_camera name="arm_thermal_cam" parent="sensor_head_mount_link">
     <!--origin xyz="${infrared_x_position} ${infrared_y_position} ${infrared_z_position}" rpy="0 0 0"/-->
-    <origin xyz="0.0345 0.0 -0.03106" rpy="0 0 0"/>
+    <origin xyz="0.0345 0.0 -0.03106" rpy="${M_PI*0.5} 0 0"/>
   </xacro:flir_a35_camera>
   <xacro:realsense_camera name="arm_rgbd_cam" parent="sensor_head_mount_link">

Commit message: Test setup with 2 LIDARs

File: hector_tracker_description/urdf/tracker_default.urdf.xacro (robot description, xacro)
@@ -165,5 +165,5 @@
     -->
     <!--Lowest box-->
-    <visual>
+<!--    <visual>
       <origin xyz="${-0.29.5} 0.115 ${0.115/2}" rpy="0 0 0"/>
       <geometry>
@@ -176,7 +176,7 @@
         <box size="${0.43-0.16} 0.15 0.115"/>
       </geometry>
-    </collision>
+    </collision>-->
     <!--Middle box-->
-    <visual>
+<!--    <visual>
       <origin xyz="${-0.34} 0.115 ${0.215+0.25*0.5}" rpy="0 0 0"/>
       <geometry>
@@ -189,5 +189,5 @@
         <box size="${0.43-0.25} 0.15 0.45"/>
       </geometry>
-    </collision>
+    </collision>  -->
     <!--
     40.8 from ref point to back of alum. frame - 12.3 (11.7 to 12.9 rotation shaft)
@@ -254,5 +254,7 @@
   <xacro:tracker_spinning_lidar_mount_macro parent="base_link"  name="spin_lidar" scaling="0.001">
     <origin xyz="-0.285 0.14 0.627" rpy="0.05 ${-M_PI*0.485} ${M_PI-0.9}"/>
-    <origin xyz="-0.025 0.0 0.0" rpy="0.0 ${M_PI*0.75} 0.0"/>
+    <!--<origin xyz="0.095 0.0 0.0225" rpy="0.0 ${M_PI*0.75} 0.0"/>-->
+    <origin xyz="0.075 0.0 0.0225" rpy="${M_PI*0.5} 0.0 ${M_PI*0.75}"/>
+    <origin xyz="-0.025 0.0 -0.0225" rpy="0.0 ${M_PI*1} ${-M_PI*0.5}"/>
   </xacro:tracker_spinning_lidar_mount_macro>
   <gazebo>

Commit message: Downward facing LIDAR for SLAM testing

File: hector_tracker_description/urdf/tracker_default.urdf.xacro (robot description, xacro)
@@ -2,7 +2,4 @@
 <robot name="taurob_tracker"
        xmlns:xacro="http://playerstage.sourceforge.net/gazebo/xmlschema/#interface">
-  <xacro:property name="flipper_offset_x" value="0.205" />
-  <xacro:property name="flipper_offset_y" value="0.15" />
-  <xacro:property name="flipper_offset_z" value="0.099" />
   <xacro:property name="M_PI" value="3.14159" />
   <xacro:property name="angle_deg" value="45" />
@@ -255,5 +252,5 @@
     <origin xyz="-0.285 0.14 0.627" rpy="0.05 ${-M_PI*0.485} ${M_PI-0.9}"/>
     <!--<origin xyz="0.095 0.0 0.0225" rpy="0.0 ${M_PI*0.75} 0.0"/>-->
-    <origin xyz="0.075 0.0 0.0225" rpy="${M_PI*0.5} 0.0 ${M_PI*0.75}"/>
+    <origin xyz="0.075 0.0 0.0225" rpy="${M_PI*0.5} 0.0 ${M_PI*1}"/>
     <origin xyz="-0.025 0.0 -0.0225" rpy="0.0 ${M_PI*1} ${-M_PI*0.5}"/>
   </xacro:tracker_spinning_lidar_mount_macro>
