Commit message: Split up model into pieces

File: hector_tracker_description/urdf/tracker_default.urdf.xacro (robot description, xacro)
@@ -2,13 +2,10 @@
 <robot name="taurob_tracker"
        xmlns:xacro="http://playerstage.sourceforge.net/gazebo/xmlschema/#interface">
-  <xacro:property name="flipper_offset_x" value="0.205" />
-  <xacro:property name="flipper_offset_y" value="0.15" />
-  <xacro:property name="flipper_offset_z" value="0.099" />
-  <xacro:property name="M_PI" value="3.14159" />
-  <xacro:property name="angle_deg" value="45" />
   <!--Required to quickly work around bug in collada_urdf (https://github.com/ros/robot_model/issues/132)-->
   <xacro:property name="box_scale_factor" value="1.0" />
   <xacro:include filename="$(find taurob_tracker_description)/urdf/tracker_chassis.urdf.xacro.xml" />
   <xacro:tracker_chassis_macro />
+  <xacro:include filename="$(find taurob_tracker_description)/urdf/tracker_chassis_cameras.urdf.xacro.xml" />
+  <xacro:tracker_chassis_cameras_macro />
   <!--Examples of adding additional robot parts below-->
   <xacro:include filename="$(find taurob_arm_description)/urdf/taurob_arm_collision_geoms_simple.urdf.xacro.xml" />
@@ -17,250 +14,11 @@
     <origin xyz="0.12 0 0.185" rpy="0 0 ${M_PI/2}"/>
   </xacro:taurob_arm_with_gripper_macro >
-  <!--<xacro:include filename="$(find hector_xacro_tools)/urdf/sensor_macros.urdf.xacro"/>-->
-  <xacro:include filename="$(find hector_sensors_description)/urdf/thermaleye_camera.urdf.xacro"/>
-  <xacro:include filename="$(find hector_sensors_description)/urdf/flir_a35_camera.urdf.xacro"/>
-  <xacro:include filename="$(find hector_sensors_description)/urdf/realsense_camera.urdf.xacro"/>
-  <xacro:include filename="$(find hector_sensors_description)/urdf/generic_camera.urdf.xacro"/>
-  <xacro:include filename="$(find hector_sensors_description)/urdf/hokuyo_utm30lx.urdf.xacro" />
-  <xacro:include filename="$(find hector_components_description)/urdf/vision_box_common.gazebo.xacro" />
-  <xacro:include filename="$(find hector_components_description)/urdf/vision_box_common_dimensions.urdf.xacro" />
-  <xacro:include filename="$(find hector_components_description)/urdf/vision_box_dimensions_hector2.urdf.xacro" />
-  <joint name="sensor_head_yaw_joint" type="revolute">
-    <origin xyz="-0.03 ${0.0565} 0.089" rpy="0 0 0"/>
-    <parent link="arm_link_3"/>
-    <child link="sensor_head_yaw_link"/>
-    <axis xyz="0 0 1"/>
-    <limit lower="${-M_PI*3/4}" upper="${M_PI*3/4}" effort="100" velocity="100"/>
-  </joint>
-  <link name="sensor_head_yaw_link">
-    <xacro:inertial_sphere mass="0.1" diameter="0.07"/>
-    <visual>
-      <origin xyz="0.0 0.0 ${cameraYawServo_size_z/2}" rpy="0 0 0"/>
-      <geometry>
-        <box size="${cameraYawServo_size_x} ${cameraYawServo_size_y} ${cameraYawServo_size_z}"/>
-      </geometry>
-      <material name="Blue"/>
-    </visual>
-    <collision>
-      <origin xyz="0.0 0.0 ${cameraYawServo_size_z/2}" rpy="0 0 0"/>
-      <geometry>
-        <box size="${cameraYawServo_size_x} ${cameraYawServo_size_y} ${cameraYawServo_size_z}"/>
-      </geometry>
-    </collision>
-  </link>
-  <joint name="sensor_head_pitch_joint" type="revolute">
-    <origin xyz="0 -0.0235 0.0921" rpy="${-M_PI/2} 0 0"/>
-    <parent link="sensor_head_yaw_link"/>
-    <child link="sensor_head_mount_link"/>
-    <axis xyz="0 0 1"/>
-    <limit lower="${-M_PI/2}" upper="${M_PI/2}" effort="100" velocity="100"/>
-  </joint>
-  <link name="sensor_head_mount_link">
-    <xacro:inertial_sphere mass="0.05" diameter="0.07"/>
-  </link>
-  <gazebo reference="sensor_head_yaw_link">
-    <material>Gazebo/Grey</material>
-  </gazebo>
-  <gazebo reference="sensor_head_mount_link">
-    <material>Gazebo/Grey</material>
-  </gazebo>
-  <xacro:include filename="$(find hector_xacro_tools)/urdf/joint_macros.urdf.xacro" />
-  <xacro:joint_standard_transmission name="sensor_head_yaw_joint"/>
-  <xacro:joint_standard_transmission name="sensor_head_pitch_joint"/>
-  <gazebo>
-    <!-- ros_control plugin -->
-    <plugin name="gazebo_ros_control_select_joints" filename="libgazebo_ros_control_select_joints.so">
-      <robotNamespace>sensor_head_control</robotNamespace>
-      <joints>sensor_head_yaw_joint sensor_head_pitch_joint</joints>
-    </plugin>
-  </gazebo>
-  <joint name="stab_laser_roll_joint" type="revolute">
-    <origin xyz="${-0.007} -0.046 ${0.078}" rpy="0 0 ${-M_PI/2}"/>
-    <parent link="arm_link_0"/>
-    <child link="stab_laser_roll_link"/>
-    <axis xyz="1 0 0"/>
-    <limit lower="${-M_PI/2}" upper="${M_PI/2}" effort="100" velocity="100"/>
-  </joint>
-  <link name="stab_laser_roll_link">
-    <xacro:inertial_sphere mass="0.1" diameter="0.07"/>
-    <visual>
-      <origin xyz="${laser1RollServo_size_x/2} 0.0 0.0" rpy="0 0 0"/>
-      <geometry>
-        <box size="${laser1RollServo_size_x} ${laser1RollServo_size_y} ${laser1RollServo_size_z}"/>
-      </geometry>
-      <material name="Blue"/>
-    </visual>
-    <collision>
-      <origin xyz="${laser1RollServo_size_x/2} 0.0 0.0" rpy="0 0 0"/>
-      <geometry>
-        <box size="${laser1RollServo_size_x} ${laser1RollServo_size_y} ${laser1RollServo_size_z}"/>
-      </geometry>
-    </collision>
-  </link>
-  <joint name="stab_laser_pitch_joint" type="revolute">
-    <origin xyz="${laser1RollServo_size_x} 0 0" rpy="0 0 0"/>
-    <parent link="stab_laser_roll_link"/>
-    <child link="stab_laser_pitch_link"/>
-    <axis xyz="0 1 0"/>
-    <limit lower="${-M_PI/2}" upper="${M_PI/2}" effort="100" velocity="100"/>
-  </joint>
-  <link name="stab_laser_pitch_link">
-    <xacro:inertial_sphere mass="0.1" diameter="0.07"/>
-    <visual>
-      <origin xyz="0.0 0.0 ${laser1_size_z/2}" rpy="0 0 0"/>
-      <geometry>
-        <!--<box size="${laser1_size_x} ${laser1_size_y} ${laser1_size_z}" /> -->
-        <box size="${laser1_size_x} ${laser1_size_y} 0.01"/>
-      </geometry>
-      <material name="Grey"/>
-    </visual>
-    <collision>
-      <origin xyz="0.0 0.0 ${laser1_size_z/2}" rpy="0 0 0"/>
-      <geometry>
-        <!--<box size="${laser1_size_x} ${laser1_size_y} ${laser1_size_z}" />-->
-        <box size="${laser1_size_x} ${laser1_size_y} 0.01"/>
-      </geometry>
-    </collision>
-  </link>
-  <gazebo reference="stab_laser_roll_link">
-    <material>Gazebo/Grey</material>
-  </gazebo>
-  <gazebo reference="stab_laser_pitch_joint">
-    <material>Gazebo/Grey</material>
-  </gazebo>
-  <xacro:joint_standard_transmission name="stab_laser_roll_joint"/>
-  <xacro:joint_standard_transmission name="stab_laser_pitch_joint"/>
-  <xacro:hokuyo_utm30lx name="stab_laser" parent="stab_laser_pitch_link" ros_topic="/stab_laser/scan_gazebo" update_rate="40" ray_count="1081" min_angle="135" max_angle="-135">
-    <origin xyz="${laser1_center_x_offset} 0 ${laser1_plane_height}" rpy="0 0 0"/>
-  </xacro:hokuyo_utm30lx>
-  <gazebo>
-    <!-- ros_control plugin -->
-    <plugin name="gazebo_ros_control_select_joints" filename="libgazebo_ros_control_select_joints.so">
-      <robotNamespace>stab_laser_control</robotNamespace>
-      <joints>stab_laser_roll_joint stab_laser_pitch_joint</joints>
-    </plugin>
-  </gazebo>
-  <joint name="structure_addon_joint" type="fixed">
-    <origin xyz="0 0 ${0.185}" rpy="0 0 0"/>
-    <parent link="base_link"/>
-    <child link="structure_addons_link"/>
-  </joint>
-  <link name="structure_addons_link">
-    <xacro:inertial_cube mass="0.1" diameter="0.07"/>
-    <!--<visual>
-      <origin xyz="-0.0 0.0 0.0" rpy="0 0 0"/>
-      <geometry>
-        <box size="${0.20 * box_scale_factor} ${0.1 * box_scale_factor} ${0.2 * box_scale_factor}"/>
-      </geometry>
-      <material name="Red">
-        <color rgba="0.6 0.0 0.0 1"/>
-      </material>
-    </visual>
-    <collision>
-      <origin xyz="-0.0 0.0 0.0" rpy="0 0 0"/>
-      <geometry>
-        <box size="0.20 0.1 0.2"/>
-      </geometry>
-    </collision>
-    -->
-    <!--Lowest box-->
-    <visual>
-      <origin xyz="${-0.29.5} 0.115 ${0.115/2}" rpy="0 0 0"/>
-      <geometry>
-        <box size="${0.43-0.16} 0.15 0.115"/>
-      </geometry>
-    </visual>
-    <collision>
-      <origin xyz="${-0.29.5} 0.115 ${0.115/2}" rpy="0 0 0"/>
-      <geometry>
-        <box size="${0.43-0.16} 0.15 0.115"/>
-      </geometry>
-    </collision>
-    <!--Middle box-->
-    <visual>
-      <origin xyz="${-0.34} 0.115 ${0.215+0.25*0.5}" rpy="0 0 0"/>
-      <geometry>
-        <box size="${0.43-0.25} 0.15 0.45"/>
-      </geometry>
-    </visual>
-    <collision>
-      <origin xyz="${-0.34} 0.115 ${0.215+0.25*0.5}" rpy="0 0 0"/>
-      <geometry>
-        <box size="${0.43-0.25} 0.15 0.45"/>
-      </geometry>
-    </collision>
-    <!--
-    40.8 from ref point to back of alum. frame - 12.3 (11.7 to 12.9 rotation shaft)
-    27.6 to top of alum. platform + 16.6 for lidar center
-    -->
-    <!--Antenna-->
-    <visual>
-      <origin xyz="${-0.38} -0.175 0.11" rpy="0 0 0"/>
-      <geometry>
-        <cylinder radius="0.015" length="0.22" />
-      </geometry>
-    </visual>
-    <collision>
-      <origin xyz="${-0.38} -0.175 0.11" rpy="0 0 0"/>
-      <geometry>
-        <cylinder radius="0.0175" length="0.22" />
-      </geometry>
-    </collision>
-  </link>
-  <gazebo reference="structure_addons_link">
-    <material>Gazebo/Grey</material>
-  </gazebo>
-    <!-- TODO: Same note as applies to imu_link -->
-  <link name="navsat_link">
-    <!--
-    <visual>
-      <geometry>
-        <cylinder radius="0.026" length="0.016" />
-      </geometry>
-      <origin xyz="0 0 0.008" />
-      <material name="black" />
-    </visual>
-    -->
-  </link>
-  <joint name="navsat_joint" type="fixed">
-    <parent link="base_link" />
-    <child link="navsat_link" />
-    <origin xyz="${-0.35.5} 0.115 ${0.68}" rpy="0 0 0"/>
-  </joint>
-  <gazebo>
-    <plugin name="gps_controller" filename="libhector_gazebo_ros_gps.so">
-      <updateRate>5</updateRate>
-      <robotNamespace>/</robotNamespace>
-      <bodyName>navsat_link</bodyName>
-      <frameId>navsat_link</frameId>
-      <topicName>/gps/fix</topicName>
-      <velocityTopicName>/gps/vel</velocityTopicName>
-      <referenceLatitude>50.396144</referenceLatitude>
-      <referenceLongitude>8.546144</referenceLongitude>
-      <referenceHeading>0</referenceHeading>
-      <referenceAltitude>0</referenceAltitude>
-      <drift>0.0001 0.0001 0.0001</drift>
-    </plugin>
-  </gazebo>
-  <xacro:flir_a35_camera name="arm_thermal_cam" parent="sensor_head_mount_link">
-    <!--origin xyz="${infrared_x_position} ${infrared_y_position} ${infrared_z_position}" rpy="0 0 0"/-->
-    <origin xyz="0.0345 0.0 -0.03106" rpy="${M_PI*0.5} 0 0"/>
-  </xacro:flir_a35_camera>
-  <xacro:realsense_camera name="arm_rgbd_cam" parent="sensor_head_mount_link">
-    <origin xyz="0.01 -0.048  ${0.01373-0.051}" rpy="${M_PI*0.5} ${kinect_pitch_position} ${kinect_yaw_position}"/>
-  </xacro:realsense_camera>
-  <!-- <xacro:vision_box_common_gazebo_plugins/> -->
-  <xacro:include filename="$(find hector_tracker_description)/urdf/tracker_spinning_lidar_mount.urdf.xacro.xml" />
-  <xacro:tracker_spinning_lidar_mount_macro parent="base_link"  name="spin_lidar" scaling="0.001">
-    <origin xyz="-0.285 0.14 0.627" rpy="0.05 ${-M_PI*0.485} ${M_PI-0.9}"/>
-    <origin xyz="-0.025 0.0 0.0" rpy="0.0 ${M_PI*0.75} 0.0"/>
-  </xacro:tracker_spinning_lidar_mount_macro>
-  <gazebo>
-    <!-- ros_control plugin -->
-    <plugin name="gazebo_ros_control_select_joints" filename="libgazebo_ros_control_select_joints.so">
-      <robotNamespace>spin_lidar_control</robotNamespace>
-      <joints>spin_lidar_spin_joint</joints>
-    </plugin>
-  </gazebo>
+  <xacro:include filename="$(find hector_tracker_description)/urdf/tracker_sensor_head.urdf.xacro.xml" />
+  <xacro:tracker_sensor_head_macro />
+  <xacro:include filename="$(find hector_tracker_description)/urdf/tracker_stab_laser.urdf.xacro.xml" />
+  <xacro:tracker_stab_laser_macro />
+  <xacro:include filename="$(find hector_tracker_description)/urdf/tracker_structure_addons.urdf.xacro.xml" />
+  <xacro:tracker_structure_addons_macro />
+  <!--
   <xacro:generic_camera name="left" parent="base_link" ros_topic="image_mono" cam_info_topic="camera_info" update_rate="10" res_x="640" res_y="480" image_format="L8" hfov="120">
     <origin xyz="${-0.285-0.17} ${0.14+0.05} ${0.627-0.11}" rpy="0 0 2.35619"/>
@@ -268,11 +26,6 @@
   <xacro:generic_camera name="right" parent="base_link" ros_topic="image_mono" cam_info_topic="camera_info" update_rate="10" res_x="640" res_y="480" image_format="L8" hfov="120">
     <origin xyz="${-0.285-0.17} ${0.14-0.05} ${0.627-0.11}" rpy="0 0 -2.35619"/>
-  </xacro:generic_camera> -->
-  <xacro:generic_camera name="front_chassis_cam" parent="base_link" ros_topic="image_raw" cam_info_topic="camera_info" update_rate="10" res_x="640" res_y="480" image_format="R8G8B8" hfov="120">
-    <origin xyz="${0.1+0.122} 0.0 0.11" rpy="0 0 0"/>
   </xacro:generic_camera>
-  <xacro:generic_camera name="rear_chassis_cam" parent="base_link" ros_topic="image_raw" cam_info_topic="camera_info" update_rate="10" res_x="640" res_y="480" image_format="R8G8B8" hfov="120">
-    <origin xyz="${-0.59+0.122} 0.0 0.11" rpy="0 0 ${M_PI}"/>
-  </xacro:generic_camera>
+  -->
   <xacro:generic_camera name="gripper_cam" parent="arm_link_4" ros_topic="image_raw" cam_info_topic="camera_info" update_rate="10" res_x="640" res_y="480" image_format="R8G8B8" hfov="80">
     <origin xyz="0 0.0 0.0" rpy="0 0 0"/>

Commit message: added 3 chilitags to robot for testing

File: hector_tracker_description/urdf/tracker_default.urdf.xacro (robot description, xacro)
@@ -14,4 +14,15 @@
     <origin xyz="0.12 0 0.185" rpy="0 0 ${M_PI/2}"/>
   </xacro:taurob_arm_with_gripper_macro >
+  <!-- ar tags -->
+  <xacro:include filename="$(find vigir_ar_alvar_description)/urdf/artag.urdf.xacro" />
+  <xacro:artag name="chilitag1" parent="base_link">
+    <origin xyz="-0.3 -0.07 0.2" rpy="0 0 0" />
+  </xacro:artag>
+  <xacro:artag name="chilitag2" parent="base_link">
+    <origin xyz="-0.1 -0.07 0.2" rpy="0 0 0" />
+  </xacro:artag>
+  <xacro:artag name="chilitag3" parent="base_link">
+    <origin xyz="-0.2 -0.03 0.2" rpy="0 0 0" />
+  </xacro:artag>
   <xacro:include filename="$(find hector_tracker_description)/urdf/tracker_sensor_head.urdf.xacro.xml" />
   <xacro:tracker_sensor_head_macro />

Commit message: positioned tags like on real robot

File: hector_tracker_description/urdf/tracker_default.urdf.xacro (robot description, xacro)
@@ -17,12 +17,12 @@
   <xacro:include filename="$(find hector_chilitag_description)/urdf/chilitag.urdf.xacro" />
   <xacro:artag name="chilitag1" parent="base_link">
-    <origin xyz="-0.3 -0.07 0.2" rpy="0 0 0" />
+    <origin xyz="-0.02 0.12 0.185" rpy="0 0 ${M_PI}" />
   </xacro:artag>
-  <xacro:artag name="chilitag2" parent="base_link">
-    <origin xyz="-0.1 -0.07 0.2" rpy="0 0 0" />
+  <xacro:artag name="chilitag0" parent="base_link">
+    <origin xyz="-0.071 -0.02 0.185" rpy="0 0 ${M_PI}" />
   </xacro:artag>
-  <xacro:artag name="chilitag3" parent="base_link">
+  <!--<xacro:artag name="chilitag3" parent="base_link">
     <origin xyz="-0.2 -0.03 0.2" rpy="0 0 0" />
-  </xacro:artag>
+  </xacro:artag>-->
   <xacro:include filename="$(find hector_tracker_description)/urdf/tracker_sensor_head.urdf.xacro.xml" />
   <xacro:tracker_sensor_head_macro />

Commit message: modified errorneous urdf to match correct model again

File: hector_tracker_description/urdf/tracker_default.urdf.xacro (robot description, xacro)
@@ -16,9 +16,9 @@
   <!-- ar tags -->
   <xacro:include filename="$(find hector_chilitag_description)/urdf/chilitag.urdf.xacro" />
+  <xacro:artag name="chilitag0" parent="base_link">
+    <origin xyz="-0.071 -0.02 0.185" rpy="0 0 ${M_PI}" />
+  </xacro:artag>
   <xacro:artag name="chilitag1" parent="base_link">
     <origin xyz="-0.02 0.12 0.185" rpy="0 0 ${M_PI}" />
-  </xacro:artag>
-  <xacro:artag name="chilitag0" parent="base_link">
-    <origin xyz="-0.071 -0.02 0.185" rpy="0 0 ${M_PI}" />
   </xacro:artag>
   <!--<xacro:artag name="chilitag3" parent="base_link">

Commit message: Fixed arm origin to match new arm updates in tracker common

File: hector_tracker_description/urdf/tracker_default.urdf.xacro (robot description, xacro)
@@ -12,5 +12,5 @@
   <xacro:include filename="$(find taurob_arm_description)/urdf/taurob_arm_macros.urdf.xacro.xml" />
   <xacro:taurob_arm_with_gripper_macro parent="base_link">
-    <origin xyz="0.12 0 0.185" rpy="0 0 ${M_PI/2}"/>
+    <origin xyz="0.12 0 0.24238" rpy="0 0 ${M_PI/2}"/>
   </xacro:taurob_arm_with_gripper_macro >
   <xacro:include filename="$(find hector_tracker_description)/urdf/tracker_sensor_head.urdf.xacro.xml" />
